Commit message: making xacro-based srdf work with end-effectors

File: barrett_wam_moveit_config/config/arm.srdf.xacro (robot description, xacro)
@@ -5,63 +5,69 @@
 -->
 <robot xmlns:xacro="http://www.ros.org/wiki/xacro">
-    <!--GROUPS: Representation of a set of joints and links. This can be useful for specifying DOF to plan for, defining arms, end effectors, etc-->
-    <!--LINKS: When a link is specified, the parent joint of that link (if it exists) is automatically included-->
-    <!--JOINTS: When a joint is specified, the child link of that joint (which will always exist) is automatically included-->
-    <!--CHAINS: When a chain is specified, all the links along the chain (including endpoints) are included in the group. Additionally, all the joints that are parents to included links are also included. This means that joints along the chain and the parent joint of the base link are included in the group-->
-    <!--SUBGROUPS: Groups can also be formed by referencing to already defined group names-->
-    <xacro:macro name="wam_7dof" params="prefix">
-      <group name="arm">
-          <joint name="${prefix}/wam_fixed_joint" />
-          <joint name="${prefix}/base_yaw_joint" />
-          <joint name="${prefix}/shoulder_pitch_joint" />
-          <joint name="${prefix}/shoulder_yaw_joint" />
-          <joint name="${prefix}/elbow_pitch_joint" />
-          <joint name="${prefix}/wrist_yaw_joint" />
-          <joint name="${prefix}/wrist_pitch_joint" />
-          <joint name="${prefix}/palm_yaw_joint" />
-          <joint name="${prefix}/wrist_palm_stump_joint" />
-      </group>
-      <!--GROUP STATES: Purpose: Define a named state for a particular group, in terms of joint values. This is useful to define states like 'folded arms'-->
-      <group_state name="zero" group="arm">
-          <joint name="${prefix}/base_yaw_joint" value="0" />
-          <joint name="${prefix}/elbow_pitch_joint" value="0" />
-          <joint name="${prefix}/palm_yaw_joint" value="0" />
-          <joint name="${prefix}/shoulder_pitch_joint" value="0" />
-          <joint name="${prefix}/shoulder_yaw_joint" value="0" />
-          <joint name="${prefix}/wrist_pitch_joint" value="0" />
-          <joint name="${prefix}/wrist_yaw_joint" value="0" />
-      </group_state>
-      <group_state name="home" group="arm">
-          <joint name="${prefix}/base_yaw_joint" value="0" />
-          <joint name="${prefix}/elbow_pitch_joint" value="3.1415" />
-          <joint name="${prefix}/palm_yaw_joint" value="1.5707" />
-          <joint name="${prefix}/shoulder_pitch_joint" value="-1.5707" />
-          <joint name="${prefix}/shoulder_yaw_joint" value="0" />
-          <joint name="${prefix}/wrist_pitch_joint" value="-1.5707" />
-          <joint name="${prefix}/wrist_yaw_joint" value="0" />
-      </group_state>
-      <!--END EFFECTOR: Purpose: Represent information about an end effector.-->
-      <end_effector name="${prefix}_palm" parent_link="${prefix}/wrist_palm_link" group="arm"/>
-      <end_effector name="${prefix}_palm_stump" parent_link="${prefix}/wrist_palm_stump_link" group="arm"/>
-      <!--DISABLE COLLISIONS: By default it is assumed that any link of the robot could potentially come into collision with any other link in the robot. This tag disables collision checking between a specified pair of links. -->
-      <disable_collisions link1="${prefix}/base_link" link2="${prefix}/forearm_link" reason="Never" />
-      <disable_collisions link1="${prefix}/base_link" link2="${prefix}/shoulder_pitch_link" reason="Never" />
-      <disable_collisions link1="${prefix}/base_link" link2="${prefix}/shoulder_yaw_link" reason="Adjacent" />
-      <disable_collisions link1="${prefix}/base_link" link2="${prefix}/upper_arm_link" reason="User" />
-      <disable_collisions link1="${prefix}/forearm_link" link2="${prefix}/shoulder_pitch_link" reason="Never" />
-      <disable_collisions link1="${prefix}/forearm_link" link2="${prefix}/shoulder_yaw_link" reason="Never" />
-      <disable_collisions link1="${prefix}/forearm_link" link2="${prefix}/upper_arm_link" reason="Adjacent" />
-      <disable_collisions link1="${prefix}/forearm_link" link2="${prefix}/wrist_pitch_link" reason="Never" />
-      <disable_collisions link1="${prefix}/forearm_link" link2="${prefix}/wrist_yaw_link" reason="Adjacent" />
-      <disable_collisions link1="${prefix}/shoulder_pitch_link" link2="${prefix}/shoulder_yaw_link" reason="Adjacent" />
-      <disable_collisions link1="${prefix}/shoulder_pitch_link" link2="${prefix}/upper_arm_link" reason="Adjacent" />
-      <disable_collisions link1="${prefix}/shoulder_pitch_link" link2="${prefix}/wrist_pitch_link" reason="Never" />
-      <disable_collisions link1="${prefix}/shoulder_pitch_link" link2="${prefix}/wrist_yaw_link" reason="Never" />
-      <disable_collisions link1="${prefix}/shoulder_yaw_link" link2="${prefix}/upper_arm_link" reason="User" />
-      <disable_collisions link1="${prefix}/shoulder_yaw_link" link2="${prefix}/wrist_pitch_link" reason="Never" />
-      <disable_collisions link1="${prefix}/shoulder_yaw_link" link2="${prefix}/wrist_yaw_link" reason="Never" />
-      <disable_collisions link1="${prefix}/upper_arm_link" link2="${prefix}/wrist_pitch_link" reason="Never" />
-      <disable_collisions link1="${prefix}/upper_arm_link" link2="${prefix}/wrist_yaw_link" reason="Never" />
-      <disable_collisions link1="${prefix}/wrist_pitch_link" link2="${prefix}/wrist_yaw_link" reason="Adjacent" />
-    </xacro:macro>
+  <!--GROUPS: Representation of a set of joints and links. This can be useful for specifying DOF to plan for, defining arms, end effectors, etc-->
+  <!--LINKS: When a link is specified, the parent joint of that link (if it exists) is automatically included-->
+  <!--JOINTS: When a joint is specified, the child link of that joint (which will always exist) is automatically included-->
+  <!--CHAINS: When a chain is specified, all the links along the chain (including endpoints) are included in the group. Additionally, all the joints that are parents to included links are also included. This means that joints along the chain and the parent joint of the base link are included in the group-->
+  <!--SUBGROUPS: Groups can also be formed by referencing to already defined group names-->
+  <xacro:macro name="wam_7dof_joints" params="prefix">
+    <joint name="${prefix}/wam_fixed_joint" />
+    <joint name="${prefix}/base_yaw_joint" />
+    <joint name="${prefix}/shoulder_pitch_joint" />
+    <joint name="${prefix}/shoulder_yaw_joint" />
+    <joint name="${prefix}/elbow_pitch_joint" />
+    <joint name="${prefix}/wrist_yaw_joint" />
+    <joint name="${prefix}/wrist_pitch_joint" />
+    <joint name="${prefix}/palm_yaw_joint" />
+  </xacro:macro>
+  <xacro:macro name="wam_7dof_states" params="prefix">
+    <!--GROUP STATES: Purpose: Define a named state for a particular group, in terms of joint values. This is useful to define states like 'folded arms'-->
+    <group_state name="zero" group="arm">
+        <joint name="${prefix}/base_yaw_joint" value="0" />
+        <joint name="${prefix}/elbow_pitch_joint" value="0" />
+        <joint name="${prefix}/palm_yaw_joint" value="0" />
+        <joint name="${prefix}/shoulder_pitch_joint" value="0" />
+        <joint name="${prefix}/shoulder_yaw_joint" value="0" />
+        <joint name="${prefix}/wrist_pitch_joint" value="0" />
+        <joint name="${prefix}/wrist_yaw_joint" value="0" />
+    </group_state>
+    <group_state name="home" group="arm">
+        <joint name="${prefix}/base_yaw_joint" value="0" />
+        <joint name="${prefix}/elbow_pitch_joint" value="3.1415" />
+        <joint name="${prefix}/palm_yaw_joint" value="1.5707" />
+        <joint name="${prefix}/shoulder_pitch_joint" value="-1.5707" />
+        <joint name="${prefix}/shoulder_yaw_joint" value="0" />
+        <joint name="${prefix}/wrist_pitch_joint" value="-1.5707" />
+        <joint name="${prefix}/wrist_yaw_joint" value="0" />
+    </group_state>
+  </xacro:macro>
+  <xacro:macro name="wam_7dof_ee_joints" params="prefix">
+    <joint name="${prefix}/wrist_palm_stump_joint" />
+  </xacro:macro>
+  <xacro:macro name="wam_7dof_ee" params="prefix">
+    <!--END EFFECTOR: Purpose: Represent information about an end effector.-->
+    <end_effector name="${prefix}_palm_stump" parent_link="${prefix}/wrist_palm_stump_link" group="arm"/>
+    <!--<end_effector name="${prefix}_palm" parent_link="${prefix}/wrist_palm_link" group="arm"/>-->
+  </xacro:macro>
+  <xacro:macro name="wam_7dof_collisions" params="prefix">
+    <!--DISABLE COLLISIONS: By default it is assumed that any link of the robot could potentially come into collision with any other link in the robot. This tag disables collision checking between a specified pair of links. -->
+    <disable_collisions link1="${prefix}/base_link" link2="${prefix}/forearm_link" reason="Never" />
+    <disable_collisions link1="${prefix}/base_link" link2="${prefix}/shoulder_pitch_link" reason="Never" />
+    <disable_collisions link1="${prefix}/base_link" link2="${prefix}/shoulder_yaw_link" reason="Adjacent" />
+    <disable_collisions link1="${prefix}/base_link" link2="${prefix}/upper_arm_link" reason="User" />
+    <disable_collisions link1="${prefix}/forearm_link" link2="${prefix}/shoulder_pitch_link" reason="Never" />
+    <disable_collisions link1="${prefix}/forearm_link" link2="${prefix}/shoulder_yaw_link" reason="Never" />
+    <disable_collisions link1="${prefix}/forearm_link" link2="${prefix}/upper_arm_link" reason="Adjacent" />
+    <disable_collisions link1="${prefix}/forearm_link" link2="${prefix}/wrist_pitch_link" reason="Never" />
+    <disable_collisions link1="${prefix}/forearm_link" link2="${prefix}/wrist_yaw_link" reason="Adjacent" />
+    <disable_collisions link1="${prefix}/shoulder_pitch_link" link2="${prefix}/shoulder_yaw_link" reason="Adjacent" />
+    <disable_collisions link1="${prefix}/shoulder_pitch_link" link2="${prefix}/upper_arm_link" reason="Adjacent" />
+    <disable_collisions link1="${prefix}/shoulder_pitch_link" link2="${prefix}/wrist_pitch_link" reason="Never" />
+    <disable_collisions link1="${prefix}/shoulder_pitch_link" link2="${prefix}/wrist_yaw_link" reason="Never" />
+    <disable_collisions link1="${prefix}/shoulder_yaw_link" link2="${prefix}/upper_arm_link" reason="User" />
+    <disable_collisions link1="${prefix}/shoulder_yaw_link" link2="${prefix}/wrist_pitch_link" reason="Never" />
+    <disable_collisions link1="${prefix}/shoulder_yaw_link" link2="${prefix}/wrist_yaw_link" reason="Never" />
+    <disable_collisions link1="${prefix}/upper_arm_link" link2="${prefix}/wrist_pitch_link" reason="Never" />
+    <disable_collisions link1="${prefix}/upper_arm_link" link2="${prefix}/wrist_yaw_link" reason="Never" />
+    <disable_collisions link1="${prefix}/wrist_pitch_link" link2="${prefix}/wrist_yaw_link" reason="Adjacent" />
+  </xacro:macro>
 </robot>

File: barrett_wam_moveit_config/config/hand.srdf.xacro (robot description, xacro)
@@ -6,26 +6,16 @@
   <!--CHAINS: When a chain is specified, all the links along the chain (including endpoints) are included in the group. Additionally, all the joints that are parents to included links are also included. This means that joints along the chain and the parent joint of the base link are included in the group-->
   <!--SUBGROUPS: Groups can also be formed by referencing to already defined group names-->
-  <xacro:macro name="bhand" params="prefix wam_prefix">
-    <group name="arm">
-      <joint name="${prefix}/bhand_base_joint" />
-      <joint name="${prefix}/finger_1/prox_joint" />
-      <joint name="${prefix}/finger_2/prox_joint" />
-      <joint name="${prefix}/finger_1/med_joint" />
-      <joint name="${prefix}/finger_2/med_joint" />
-      <joint name="${prefix}/finger_3/med_joint" />
-      <joint name="${prefix}/finger_1/dist_joint" />
-      <joint name="${prefix}/finger_2/dist_joint" />
-      <joint name="${prefix}/finger_3/dist_joint" />
-      <joint name="${prefix}/bhand_palm_surface_joint" />
-      <joint name="${prefix}/bhand_grasp_joint" />
-    </group>
+  <xacro:macro name="bhand_joints" params="prefix wam_prefix">
+    <joint name="${prefix}/bhand_base_joint" />
+    <joint name="${prefix}/bhand_grasp_joint" />
+    <link name="${prefix}/bhand_grasp_link" />
     <!--GROUP STATES: Purpose: Define a named state for a particular group, in terms of joint values. This is useful to define states like 'folded arms'-->
     <!--END EFFECTOR: Purpose: Represent information about an end effector.-->
-    <end_effector name="${prefix}_bhand_palm" parent_link="${prefix}/bhand_palm_surface_joint" group="arm"/>
-    <end_effector name="${prefix}_bhand_grasp" parent_link="${prefix}/bhand_grasp_joint" group="arm"/>
     <!--DISABLE COLLISIONS: By default it is assumed that any link of the robot could potentially come into collision with any other link in the robot. This tag disables collision checking between a specified pair of links. -->
-    <xacro:bhand_links prefix="${prefix}" wam_prefix="${wam_prefix}"/>
   </xacro:macro>
-  <xacro:macro name="bhand_links" params="prefix wam_prefix">
+  <xacro:macro name="bhand_ee" params="prefix wam_prefix">
+    <end_effector name="${wam_prefix}_bhand_grasp" parent_link="${prefix}/bhand_grasp_link" group="arm"/>
+  </xacro:macro>
+  <xacro:macro name="bhand_collisions" params="prefix wam_prefix">
     <xacro:bhand_palm prefix="${prefix}" wam_prefix="${wam_prefix}"/>
     <xacro:bhand_finger_1_or_2 prefix="${prefix}" finger="1" wam_prefix="${wam_prefix}"/>
@@ -72,6 +62,8 @@
     <disable_collisions link1="${prefix}/finger_${finger}/dist_link" link2="${wam_prefix}/wrist_palm_link" reason="Never" />
     <disable_collisions link1="${prefix}/finger_${finger}/dist_link" link2="${prefix}/bhand_palm_link" reason="Never" />
-    <disable_collisions link1="${prefix}/finger_${finger}/dist_link" link2="${prefix}/finger_${finger}/prox_link" reason="Never" />
     <disable_collisions link1="${prefix}/finger_${finger}/dist_link" link2="${prefix}/finger_${finger}/med_link" reason="Adjacent" />
+    <xacro:if value="${prox}">
+      <disable_collisions link1="${prefix}/finger_${finger}/dist_link" link2="${prefix}/finger_${finger}/prox_link" reason="Never" />
+    </xacro:if>
   </xacro:macro>
 </robot>

File: barrett_wam_moveit_config/config/wam7.srdf.xacro (robot description, xacro)
@@ -2,10 +2,43 @@
 <robot xmlns:xacro="http://www.ros.org/wiki/xacro" name="wam">
   <xacro:include filename="$(find barrett_wam_moveit_config)/config/wam_top.srdf.xacro"/>
-  <xacro:wam_7dof prefix="$(arg prefix)"/>
+  <!-- The "arm" group.
+       This is the group used for motion planning. We have to compose a single
+       group because MoveIt does not allow combining of multiple group
+       specifications with the same name. Additionally, in order to work
+       with the planner, the motion planning group needs to be a chain, and
+       can't have a more general tree structure. -->
+  <group name="arm">
+    <!-- Include the basic WAM joints -->
+    <xacro:wam_7dof_joints prefix="$(arg prefix)"/>
+    <!-- Include an additional joint for the "empty" end-effector -->
+    <xacro:if value="$(arg empty)">
+      <xacro:wam_7dof_ee_joints prefix="$(arg prefix)"/>
+    </xacro:if>
+    <!-- Include the semantic description of the hand links -->
+    <xacro:if value="$(arg hand)">
+      <xacro:bhand_joints prefix="$(arg prefix)/hand" wam_prefix="$(arg prefix)"/>
+    </xacro:if>
+    <!-- Include the semantic description of the ball links -->
+    <xacro:if value="$(arg ball)">
+      <xacro:bball_joints prefix="$(arg prefix)/ball"/>
+    </xacro:if>
+  </group>
+  <!-- Include WAM poses -->
+  <xacro:wam_7dof_states prefix="$(arg prefix)"/>
+  <!-- Include WAM collision descriptions -->
+  <xacro:wam_7dof_collisions prefix="$(arg prefix)"/>
+  <!-- Include the specification of the "empty" end-effector -->
+  <xacro:if value="$(arg empty)">
+    <xacro:wam_7dof_ee prefix="$(arg prefix)"/>
+  </xacro:if>
+  <!-- Include the specification of the hand end-effector and collision descriptions -->
   <xacro:if value="$(arg hand)">
-    <xacro:bhand prefix="$(arg prefix)/hand" wam_prefix="$(arg prefix)"/>
+    <xacro:bhand_ee prefix="$(arg prefix)/hand" wam_prefix="$(arg prefix)"/>
+    <xacro:bhand_collisions prefix="$(arg prefix)/hand" wam_prefix="$(arg prefix)"/>
   </xacro:if>
+  <!-- Include the specification of the ball end-effector and collision descriptions -->
   <xacro:if value="$(arg ball)">
-    <xacro:bball prefix="$(arg prefix)/ball"/>
+    <xacro:bball_ee prefix="$(arg prefix)/ball"/>
+    <xacro:bball_collisions prefix="$(arg prefix)/ball"/>
   </xacro:if>
 </robot>
