Commit message: updating ball srdf with proper collision flags

File: barrett_wam_moveit_config/config/ball.srdf.xacro (robot description, xacro)
@@ -16,5 +16,9 @@
   </xacro:macro>
   <xacro:macro name="bball_ee" params="prefix wam_prefix">
-    <end_effector name="${wam_prefix}_bball_center_link" parent_link="${prefix}/bball_center_link" group="arm"/>
+    <end_effector name="${wam_prefix}_bball_center" parent_link="${prefix}/bball_center_link" group="arm"/>
+  </xacro:macro>
+  <xacro:macro name="bball_collisions" params="prefix wam_prefix">
+    <disable_collisions link1="${prefix}/bball_base_link" link2="${prefix}/bball_center_link" reason="Never" />
+    <disable_collisions link1="${prefix}/bball_base_link" link2="${wam_prefix}/wrist_yaw_link" reason="Never" />
   </xacro:macro>
 </robot>

File: barrett_wam_moveit_config/config/wam7.srdf.xacro (robot description, xacro)
@@ -40,5 +40,5 @@
   <xacro:if value="$(arg ball)">
     <xacro:bball_ee prefix="$(arg prefix)/ball" wam_prefix="$(arg prefix)"/>
-    <!--<xacro:bball_collisions prefix="$(arg prefix)/ball"/>-->
+    <xacro:bball_collisions prefix="$(arg prefix)/ball" wam_prefix="$(arg prefix)"/>
   </xacro:if>
 </robot>
