Commit message: fixing hand self-collisions

File: barrett_wam_moveit_config/config/hand.srdf.xacro (robot description, xacro)
@@ -19,17 +19,17 @@
   <xacro:macro name="bhand_collisions" params="prefix wam_prefix">
     <xacro:bhand_palm prefix="${prefix}" wam_prefix="${wam_prefix}"/>
-    <xacro:bhand_finger_1_or_2 prefix="${prefix}" finger="1" wam_prefix="${wam_prefix}"/>
-    <xacro:bhand_finger_1_or_2 prefix="${prefix}" finger="2" wam_prefix="${wam_prefix}"/>
+    <xacro:bhand_finger_1_or_2 prefix="${prefix}" finger="1" other="2" wam_prefix="${wam_prefix}"/>
+    <xacro:bhand_finger_1_or_2 prefix="${prefix}" finger="2" other="1" wam_prefix="${wam_prefix}"/>
     <xacro:bhand_finger_3 prefix="${prefix}" wam_prefix="${wam_prefix}"/>
   </xacro:macro>
   <!-- Fingers -->
-  <xacro:macro name="bhand_finger_1_or_2" params="prefix finger wam_prefix">
+  <xacro:macro name="bhand_finger_1_or_2" params="prefix finger other wam_prefix">
     <xacro:bhand_finger_prox prefix="${prefix}" finger="${finger}" wam_prefix="${wam_prefix}"/>
     <xacro:bhand_finger_med prefix="${prefix}" finger="${finger}" prox="true" wam_prefix="${wam_prefix}"/>
-    <xacro:bhand_finger_dist prefix="${prefix}" finger="${finger}" prox="true" wam_prefix="${wam_prefix}"/>
+    <xacro:bhand_finger_dist prefix="${prefix}" finger="${finger}" other_a="${other}" other_b="3" prox="true" wam_prefix="${wam_prefix}"/>
   </xacro:macro>
   <xacro:macro name="bhand_finger_3" params="prefix wam_prefix">
     <xacro:bhand_finger_med prefix="${prefix}" finger="3" prox="false" wam_prefix="${wam_prefix}"/>
-    <xacro:bhand_finger_dist prefix="${prefix}" finger="3" prox="false" wam_prefix="${wam_prefix}"/>
+    <xacro:bhand_finger_dist prefix="${prefix}" finger="3" other_a="1" other_b="2" prox="false" wam_prefix="${wam_prefix}"/>
   </xacro:macro>
   <!-- Components -->
@@ -45,4 +45,5 @@
     <disable_collisions link1="${prefix}/finger_${finger}/prox_link" link2="${wam_prefix}/wrist_palm_link" reason="Never" />
     <disable_collisions link1="${prefix}/finger_${finger}/prox_link" link2="${prefix}/bhand_palm_link" reason="Adjacent" />
+    <disable_collisions link1="${prefix}/finger_${finger}/prox_link" link2="${prefix}/finger_3/dist_link" reason="Fingers" />
   </xacro:macro>
   <xacro:macro name="bhand_finger_med" params="prefix finger prox wam_prefix">
@@ -56,5 +57,5 @@
     </xacro:if>
   </xacro:macro>
-  <xacro:macro name="bhand_finger_dist" params="prefix finger prox wam_prefix">
+  <xacro:macro name="bhand_finger_dist" params="prefix finger other_a other_b prox wam_prefix">
     <passive_joint name="${prefix}/finger_${finger}/dist_joint" />
     <disable_collisions link1="${prefix}/finger_${finger}/dist_link" link2="${wam_prefix}/wrist_yaw_link" reason="Never" />
@@ -66,4 +67,9 @@
       <disable_collisions link1="${prefix}/finger_${finger}/dist_link" link2="${prefix}/finger_${finger}/prox_link" reason="Never" />
     </xacro:if>
+    <!-- other fingers -->
+    <disable_collisions link1="${prefix}/finger_${finger}/dist_link" link2="${prefix}/finger_${other_a}/dist_link" reason="Adjacent" />
+    <disable_collisions link1="${prefix}/finger_${finger}/dist_link" link2="${prefix}/finger_${other_a}/med_link" reason="Adjacent" />
+    <disable_collisions link1="${prefix}/finger_${finger}/dist_link" link2="${prefix}/finger_${other_b}/dist_link" reason="Fingers" />
+    <disable_collisions link1="${prefix}/finger_${finger}/dist_link" link2="${prefix}/finger_${other_b}/med_link" reason="Fingers" />
   </xacro:macro>
 </robot>
